File: pcb panda display.kicad_sch (KiCad schematic)
At the start: 6 parts, among them J1 Conn_01x12_Pin, SW1 SW_Push, SW2 SW_Push, SW3 SW_Push, U1 ST7735, U2 C3 Pico

Commit message: Add files via upload
Parts:
- added H1, H2: MountingHole, MountingHole:MountingHole_2.5mm, symbol Mechanical:MountingHole
Other:
- moved on the sheet: U1
Changed lines of the file:
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@@
 	)
 	(no_connect
-		(at 76.2 109.22)
-	)
-	(no_connect
-		(at 76.2 96.52)
-	)
-	(no_connect
-		(at 76.2 101.6)
-	)
-	(no_connect
-		(at 76.2 99.06)
-	)
-	(no_connect
-		(at 76.2 106.68)
+		(at 115.57 96.52)
+	)
+	(no_connect
+		(at 115.57 83.82)
+	)
+	(no_connect
+		(at 115.57 88.9)
+	)
+	(no_connect
+		(at 115.57 86.36)
+	)
+	(no_connect
+		(at 115.57 93.98)
 	)
 	(no_connect
@@
 	)
 	(no_connect
-		(at 76.2 93.98)
-	)
-	(no_connect
-		(at 76.2 104.14)
-	)
-	(no_connect
-		(at 76.2 86.36)
-	)
-	(no_connect
-		(at 76.2 88.9)
+		(at 115.57 81.28)
+	)
+	(no_connect
+		(at 115.57 91.44)
+	)
+	(no_connect
+		(at 115.57 73.66)
+	)
+	(no_connect
+		(at 115.57 76.2)
 	)
 	(no_connect
@@
 	)
 	(no_connect
-		(at 76.2 111.76)
+		(at 115.57 99.06)
 	)
 	(no_connect
@@
 	)
 	(no_connect
-		(at 76.2 91.44)
-	)
-	(no_connect
-		(at 76.2 83.82)
+		(at 115.57 78.74)
+	)
+	(no_connect
+		(at 115.57 71.12)
 	)
 	(wire
@@
 	)
 	(symbol
+		(lib_id "Mechanical:MountingHole")
+		(at 55.88 144.78 0)
+		(unit 1)
+		(exclude_from_sim yes)
+		(in_bom no)
+		(on_board yes)
+		(dnp no)
+		(fields_autoplaced yes)
+		(property "Reference" "H1"
+			(at 58.42 143.5099 0)
+			(effects
+				(font
+					(size 1.27 1.27)
+				)
+				(justify left)
+			)
+		)
+		(property "Value" "MountingHole"
+			(at 58.42 146.0499 0)
+			(effects
+				(font
+					(size 1.27 1.27)
+				)
+				(justify left)
+			)
+		)
+		(property "Footprint" "MountingHole:MountingHole_2.5mm"
+			(at 55.88 144.78 0)
+			(effects
+				(font
+					(size 1.27 1.27)
+				)
+				(hide yes)
+			)
+		)
+		(property "Datasheet" "~"
+			(at 55.88 144.78 0)
+			(effects
+				(font
+					(size 1.27 1.27)
+				)
+				(hide yes)
+			)
+		)
+		(property "Description" "Mounting Hole without connection"
+			(at 55.88 144.78 0)
+			(effects
+				(font
+					(size 1.27 1.27)
+				)
+				(hide yes)
+			)
+		)
+		(instances
+			(project ""
+				(path "/38e71931-0e63-4a8e-9cbb-944b97ed850d"
+					(reference "H1")
+					(unit 1)
+				)
+			)
+		)
+	)
+	(symbol
 		(lib_id "power:+3.3V")
 		(at 116.84 149.86 0)
@@
 	(symbol
 		(lib_id "PhilsLibrary:ST7735")
-		(at 63.5 97.79 0)
+		(at 102.87 85.09 0)
 		(unit 1)
 		(exclude_from_sim no)
@@
 		(fields_autoplaced yes)
 		(property "Reference" "U1"
-			(at 64.135 73.66 0)
+			(at 103.505 60.96 0)
 			(effects
 				(font
@@
 		)
 		(property "Value" "ST7735"
-			(at 64.135 76.2 0)
+			(at 103.505 63.5 0)
 			(effects
 				(font
@@
 		)
 		(property "Footprint" "PhilsFootprintLibrary:Display_ST7735"
-			(at 59.69 95.25 0)
+			(at 99.06 82.55 0)
 			(effects
 				(font
@@
 		)
 		(property "Datasheet" "https://www.displayfuture.com/Display/datasheet/controller/ST7735.pdf"
-			(at 63.5 121.92 0)
+			(at 102.87 109.22 0)
 			(effects
 				(font
@@
 		)
 		(property "Description" "1.8\" 128*160 SPI TFT Display"
-			(at 63.5 97.79 0)
+			(at 102.87 85.09 0)
 			(effects
 				(font
@@
 					(unit 1)
 				)
+			)
+		)
+	)
+	(symbol
+		(lib_id "Mechanical:MountingHole")
+		(at 76.2 140.97 0)
+		(unit 1)
+		(exclude_from_sim yes)
+		(in_bom no)
+		(on_board yes)
+		(dnp no)
+		(fields_autoplaced yes)
+		(property "Reference" "H2"
+			(at 78.74 139.6999 0)
+			(effects
+				(font
+					(size 1.27 1.27)
+				)
+				(justify left)
+			)
+		)
+		(property "Value" "MountingHole"
+			(at 78.74 142.2399 0)
+			(effects
+				(font
+					(size 1.27 1.27)
+				)
+				(justify left)
+			)
+		)
+		(property "Footprint" "MountingHole:MountingHole_2.5mm"
+			(at 76.2 140.97 0)
+			(effects
+				(font
+					(size 1.27 1.27)
+				)
+				(hide yes)
+			)
+		)
+		(property "Datasheet" "~"
+			(at 76.2 140.97 0)
+			(effects
+				(font
+					(size 1.27 1.27)
+				)
+				(hide yes)
+			)
+		)
+		(property "Description" "Mounting Hole without connection"
+			(at 76.2 140.97 0)
+			(effects
+				(font
+					(size 1.27 1.27)
+				)
+				(hide yes)
+			)
+		)
+		(instances
+			(project ""
+				(path "/38e71931-0e63-4a8e-9cbb-944b97ed850d"
+					(reference "H2")
+					(unit 1)
+				)
